File: b.kicad_sch (KiCad schematic)
At the start: 0 parts

Commit message: blind ref
Other:
- added sheet r (./sch/r.kicad_sch)
Changed lines of the file:
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@@
 (kicad_sch (version 20230121) (generator eeschema)
   (paper "A4")
+  (sheet (at 156.21 95.885) (size 24.765 12.7) (fields_autoplaced)
+    (stroke (width 0.1524) (type solid))
+    (fill (color 0 0 0 0.0000))
+    (property "Sheetname" "r" (at 156.21 95.1734 0)
+      (effects (font (size 1.27 1.27)) (justify left bottom))
+    )
+    (property "Sheetfile" "./sch/r.kicad_sch" (at 156.21 109.1696 0)
+      (effects (font (size 1.27 1.27)) (justify left top))
+    )
+    (instances
+      (project "b"
+        (path "/d97b04af-f940-4b37-9b46-3257568904dc" (page "2"))
+      )
+    )
+  )
   (sheet_instances
     (path "/" (page "1"))
